Commit message: update v2.1.0

File: roch_description/robots/roch_standard.urdf.xacro (robot description, xacro)
@@ -6,5 +6,5 @@
 <robot name="roch" xmlns:xacro="http://ros.org/wiki/xacro">
   <xacro:include filename="$(find roch_description)/urdf/roch_library.urdf.xacro" />
-  <roch/>
-  <stack_standard                 parent="base_link"/>
+  <xacro:roch/>
+  <xacro:stack_standard parent="base_link"/>
 </robot>

File: roch_description/robots/roch_standard_astra.urdf.xacro (robot description, xacro)
@@ -7,6 +7,6 @@
 <robot name="roch" xmlns:xacro="http://ros.org/wiki/xacro">
   <xacro:include filename="$(find roch_description)/urdf/roch_library.urdf.xacro" />
-  <roch/>
-  <stack_standard                 parent="base_link"/>
-  <sensor_astra                   parent="base_link"/>
+  <xacro:roch/>
+  <xacro:stack_standard parent="base_link"/>
+  <xacro:sensor_astra parent="base_link"/>
 </robot>

File: roch_description/robots/roch_standard_astra_rplidar.urdf.xacro (robot description, xacro)
@@ -8,7 +8,7 @@
 <robot name="roch" xmlns:xacro="http://ros.org/wiki/xacro">
   <xacro:include filename="$(find roch_description)/urdf/roch_library.urdf.xacro" />
-  <roch/>
-  <stack_standard                 parent="base_link"/>
-  <sensor_astra                   parent="base_link"/>
-  <rplidar                        parent="base_link"/>
+  <xacro:roch/>
+  <xacro:stack_standard parent="base_link"/>
+  <xacro:sensor_astra parent="base_link"/>
+  <xacro:rplidar parent="base_link"/>
 </robot>

File: roch_description/robots/roch_standard_rplidar.urdf.xacro (robot description, xacro)
@@ -7,6 +7,6 @@
 <robot name="roch" xmlns:xacro="http://ros.org/wiki/xacro">
   <xacro:include filename="$(find roch_description)/urdf/roch_library.urdf.xacro" />
-  <roch/>
-  <stack_standard                 parent="base_link"/>
-  <rplidar                        parent="base_link"/>
+  <xacro:roch/>
+  <xacro:stack_standard parent="base_link"/>
+  <xacro:rplidar parent="base_link"/>
 </robot>

File: roch_description/urdf/roch.urdf.xacro (robot description, xacro)
@@ -5,9 +5,9 @@
   <xacro:include filename="$(find roch_description)/urdf/roch_gazebo.urdf.xacro"/>
   <xacro:include filename="$(find roch_description)/urdf/roch_sensors.urdf.xacro"/>
-  <property name="M_PI" value="3.14159"/>
+  <xacro:property name="M_PI" value="3.14159"/>
   <!-- Base Size -->
-  <property name="base_x_size" value="0.353080" />
-  <property name="base_y_size" value="0.299330" />
-  <property name="base_z_size" value="0.150000" />
+  <xacro:property name="base_x_size" value="0.353080" />
+  <xacro:property name="base_y_size" value="0.299330" />
+  <xacro:property name="base_z_size" value="0.150000" />
   <!-- Wheel Mounting Positions -->
   <xacro:property name="wheelbase" value="-0.095" />
@@ -17,6 +17,6 @@
   <xacro:property name="wheel_length" value="0.014" />
   <xacro:property name="wheel_radius" value="0.0475" />
- <!---->
- <xacro:macro name="roch">
+  <!---->
+  <xacro:macro name="roch">
     <!-- Base link is on the ground under the robot -->
     <link name="base_footprint"/>
@@ -34,12 +34,12 @@
         <origin xyz="0 0 0" rpy="0 0 0" />
         <geometry>
-	  <mesh filename="package://roch_description/meshes/chassis.dae"/>
+          <mesh filename="package://roch_description/meshes/chassis.dae"/>
         </geometry>
-       <xacro:insert_block name="roch_dark_white" />
+        <xacro:insert_block name="roch_dark_white" />
       </visual>
       <collision>
         <origin xyz="0 0 ${base_z_size*3/4}" rpy="0 0 0" />
         <geometry>
-         <box size="0.35308 .29933 .155"/>
+          <box size="0.35308 .29933 .155"/>
         </geometry>
       </collision>
@@ -61,8 +61,7 @@
       </inertial>
     </link>
-    <gazebo reference="base_link">
-    </gazebo>
-<!-- Xacro macros -->
-  <!-- roch wheel macros -->
+    <gazebo reference="base_link"/>
+    <!-- Xacro macros -->
+    <!-- roch wheel macros -->
     <xacro:roch_wheel wheel_prefix="front_left">
       <origin xyz="0 ${track/2} ${wheel_vertical_offset-0.0005}" rpy="0 0 0" />
@@ -71,6 +70,6 @@
       <origin xyz="0 ${-track/2} ${wheel_vertical_offset-0.0005}" rpy="0 0 0" />
     </xacro:roch_wheel>
-   <link name="front_wheel_link">
-    <collision>
+    <link name="front_wheel_link">
+      <collision>
         <geometry>
           <cylinder length="0.018" radius="0.0127"/>
@@ -82,10 +81,10 @@
         <origin xyz="0 0 0" />
         <inertia ixx="0.001" ixy="0.0" ixz="0.0"
-                 iyy="0.001" iyz="0.0"
-                 izz="0.001" />
+                iyy="0.001" iyz="0.0"
+                izz="0.001" />
       </inertial>
-   </link>
-   <link name="rear_wheel_link">
-    <collision>
+    </link>
+    <link name="rear_wheel_link">
+      <collision>
         <geometry>
           <cylinder length="0.018" radius="0.0127"/>
@@ -97,29 +96,29 @@
         <origin xyz="0 0 0" />
         <inertia ixx="0.001" ixy="0.0" ixz="0.0"
-                 iyy="0.001" iyz="0.0"
-                 izz="0.001" />
+                iyy="0.001" iyz="0.0"
+                izz="0.001" />
       </inertial>
-   </link>
-<!--                 modify                     -->
-<!--              range_z: -0.007 ~ -0.008      -->
-<!--        if not modify in gazebo will shack  -->
-<!--                                            -->
-<!--             Fixed this Bug                 -->
-<!--             Finally param                  -->
-<!--          L:0.13 0 -0.125                   -->
-<!--          R:-0.13 0 -0.0084                 -->
-<!--                                            -->
-   <joint name="fornt_wheel_joint" type="fixed">
+    </link>
+    <!--                 modify                     -->
+    <!--              range_z: -0.007 ~ -0.008      -->
+    <!--        if not modify in gazebo will shack  -->
+    <!--                                            -->
+    <!--             Fixed this Bug                 -->
+    <!--             Finally param                  -->
+    <!--          L:0.13 0 -0.125                   -->
+    <!--          R:-0.13 0 -0.0084                 -->
+    <!--                                            -->
+    <joint name="fornt_wheel_joint" type="fixed">
       <origin xyz="0.13 0 -0.0125 " rpy="${-M_PI/2} 0 0" />
       <parent link="base_link" />
       <child link="front_wheel_link" />
-   </joint>
-   <joint name="rear_wheel_joint" type="fixed">
+    </joint>
+    <joint name="rear_wheel_joint" type="fixed">
       <origin xyz="-0.13 0 -0.0084 " rpy="${-M_PI/2} 0 0" />
       <parent link="base_link" />
       <child link="rear_wheel_link" />
-   </joint>
-<!-- Roch sensors -->
- <!-- IMU Link is the standard mounting position for the R1371T IMU.-->
+    </joint>
+    <!-- Roch sensors -->
+    <!-- IMU Link is the standard mounting position for the R1371T IMU.-->
     <!-- Can be modified with environment variables in /etc/ros/setup.bash -->
     <link name="imu_link">
@@ -162,6 +161,6 @@
       <origin xyz="0.12695 -0.06874 0.0065" rpy="0 ${M_PI/2} 0" />
     </xacro:roch_cliff>
- <!-- roch Gazebo simulation details -->
-  <roch_robot_gazebo/>
-</xacro:macro>
+    <!-- roch Gazebo simulation details -->
+    <roch_robot_gazebo/>
+  </xacro:macro>
 </robot>

File: roch_description/urdf/roch_properties.urdf.xacro (robot description, xacro)
@@ -1,4 +1,4 @@
 <?xml version="1.0"?>
-<robot>
+<robot xmlns:xacro="http://ros.org/wiki/xacro">
   <!--
     These properties must be observed by any machine
@@ -6,5 +6,5 @@
     to the REP for more details.
     http://www.ros.org/reps/rep-0119.html
-   -->
+  -->
   <!--
    ======================================================================
@@ -18,32 +18,32 @@
      Note: REP needs to be updated with the information below
      (currently in development and awaiting feedback)
-   -->
+  -->
 <!-- asus xtion param -->
-  <property name="asus_xtion_px" value="-0.145" />
-  <property name="asus_xtion_py" value="-0.025" />
-  <property name="asus_xtion_pz" value="0.721" />
-  <property name="asus_xtion_or" value="0" />
-  <property name="asus_xtion_op" value="0" />
-  <property name="asus_xtion_oy" value="0" />
+  <xacro:property name="asus_xtion_px" value="-0.145" />
+  <xacro:property name="asus_xtion_py" value="-0.025" />
+  <xacro:property name="asus_xtion_pz" value="0.721" />
+  <xacro:property name="asus_xtion_or" value="0" />
+  <xacro:property name="asus_xtion_op" value="0" />
+  <xacro:property name="asus_xtion_oy" value="0" />
 <!-- kinect param -->
-  <property name="kinect_px" value="-0.145" />
-  <property name="kinect_py" value="-0.025" />
-  <property name="kinect_pz" value="0.721" />
-  <property name="kinect_or" value="0" />
-  <property name="kinect_op" value="0" />
-  <property name="kinect_oy" value="0" />
+  <xacro:property name="kinect_px" value="-0.145" />
+  <xacro:property name="kinect_py" value="-0.025" />
+  <xacro:property name="kinect_pz" value="0.721" />
+  <xacro:property name="kinect_or" value="0" />
+  <xacro:property name="kinect_op" value="0" />
+  <xacro:property name="kinect_oy" value="0" />
 <!-- Intel R200 param -->
-  <property name="r200_px" value="-0.135" />
-  <property name="r200_py" value="-0.065" />
-  <property name="r200_pz" value="0.7" />
-  <property name="r200_or" value="0" />
-  <property name="r200_op" value="0" />
-  <property name="r200_oy" value="0" />
+  <xacro:property name="r200_px" value="-0.135" />
+  <xacro:property name="r200_py" value="-0.065" />
+  <xacro:property name="r200_pz" value="0.7" />
+  <xacro:property name="r200_or" value="0" />
+  <xacro:property name="r200_op" value="0" />
+  <xacro:property name="r200_oy" value="0" />
 <!-- Orbbec Astra param -->
-  <property name="astra_px" value="-0.12" />
-  <property name="astra_py" value="0.0" />
-  <property name="astra_pz" value="0.715" />
-  <property name="astra_or" value="0" />
-  <property name="astra_op" value="0" />
-  <property name="astra_oy" value="0" />
+  <xacro:property name="astra_px" value="-0.12" />
+  <xacro:property name="astra_py" value="0.0" />
+  <xacro:property name="astra_pz" value="0.715" />
+  <xacro:property name="astra_or" value="0" />
+  <xacro:property name="astra_op" value="0" />
+  <xacro:property name="astra_oy" value="0" />
 </robot>

File: roch_description/urdf/sensors/astra.urdf.xacro (robot description, xacro)
@@ -13,22 +13,22 @@
     <link name="camera_link">
       <visual>
-       <origin xyz="0 0 0" rpy="1.5707963 0 1.5707963"/>
+        <origin xyz="0 0 0" rpy="1.5707963 0 1.5707963"/>
         <geometry>
-         <mesh filename="package://roch_description/meshes/sensors/astra.dae" scale="0.5 0.5 0.5" />
+          <mesh filename="package://roch_description/meshes/sensors/astra.dae" scale="0.5 0.5 0.5" />
         </geometry>
-	    <xacro:insert_block name="roch_black"/>
+      <xacro:insert_block name="roch_black"/>
       </visual>
-  	  <collision>
+      <collision>
         <origin xyz="0.0 0.0 0.0" rpy="1.5707963 0 1.5707963"/>
-  	    <geometry>.
-         <mesh filename="package://roch_description/meshes/sensors/astra.dae" scale="0.5 0.5 0.5" />
-  	    </geometry>
-  	  </collision>
+        <geometry>.
+          <mesh filename="package://roch_description/meshes/sensors/astra.dae" scale="0.5 0.5 0.5" />
+        </geometry>
+      </collision>
       <inertial>
         <mass value="0.564" />
         <origin xyz="0 0 0" />
         <inertia ixx="0.003881243" ixy="0.0" ixz="0.0"
-                 iyy="0.000498940" iyz="0.0"
-                 izz="0.003879257" />
+                  iyy="0.000498940" iyz="0.0"
+                  izz="0.003879257" />
       </inertial>
     </link>
@@ -48,18 +48,18 @@
          files. However, for Gazebo simulation we need them, so we add them here.
          (Hence, don't publish them additionally!) -->
-	<joint name="camera_depth_joint" type="fixed">
-	  <origin xyz="0 ${-0.03 -astra_cam_py} 0" rpy="0 0 0" />
-	  <parent link="camera_rgb_frame" />
-	  <child link="camera_depth_frame" />
-	</joint>
-	<link name="camera_depth_frame"/>
-	<joint name="camera_depth_optical_joint" type="fixed">
-	  <origin xyz="0 0 0" rpy="${-M_PI/2} 0 ${-M_PI/2}" />
-	  <parent link="camera_depth_frame" />
-	  <child link="camera_depth_optical_frame" />
-	</joint>
-	<link name="camera_depth_optical_frame"/>
-	<!-- astra sensor for simulation -->
-	<roch_sim_3dsensor/>
-  </xacro:macro>
+    <joint name="camera_depth_joint" type="fixed">
+      <origin xyz="0 ${-0.03 -astra_cam_py} 0" rpy="0 0 0" />
+      <parent link="camera_rgb_frame" />
+      <child link="camera_depth_frame" />
+    </joint>
+    <link name="camera_depth_frame"/>
+    <joint name="camera_depth_optical_joint" type="fixed">
+      <origin xyz="0 0 0" rpy="${-M_PI/2} 0 ${-M_PI/2}" />
+      <parent link="camera_depth_frame" />
+      <child link="camera_depth_optical_frame" />
+    </joint>
+    <link name="camera_depth_optical_frame"/>
+    <!-- astra sensor for simulation -->
+    <roch_sim_3dsensor/>
+    </xacro:macro>
 </robot>

File: roch_description/urdf/sensors/rplidar.urdf.xacro (robot description, xacro)
@@ -56,12 +56,12 @@
       </collision>
     </link>
-     <joint name="base_laser_link_mount" type="fixed">
-        <origin xyz="0.1 0 0.165" rpy="0 0 0" />
-        <parent link="${parent}" />
-        <child link="base_laser_link" />
-      </joint>
+    <joint name="base_laser_link_mount" type="fixed">
+      <origin xyz="0.1 0 0.165" rpy="0 0 0" />
+      <parent link="${parent}" />
+      <child link="base_laser_link" />
+    </joint>
     <link name="base_laser"/>
     <joint name="base_laser_joint" type="fixed">
-      <origin xyz="0 0 0.04076" rpy=" 0 0 2.2689" />
+      <origin xyz="0 0 0.04076" rpy="0 0 ${M_PI}" />  <!-- y2.2689 -->
       <parent link="base_laser_link" />
       <child link="base_laser" />

File: roch_description/urdf/stacks/standard/standard.urdf.xacro (robot description, xacro)
@@ -2,11 +2,11 @@
 <!--
   standard stacks of Roch
- -->
+-->
 <robot name="stack_standard" xmlns:xacro="http://ros.org/wiki/xacro">
   <xacro:include filename="$(find roch_description)/urdf/common_properties.urdf.xacro"/>
   <!-- hexagons for roch -->
-    <!-- Xacro properties -->
+  <!-- Xacro properties -->
   <xacro:property name="M_SCALE" value="0.001"/>
-<!-- Xacro macros -->
+  <!-- Xacro macros -->
   <!-- Pole bottom macros -->
   <xacro:macro name="stack_bottom_pole" params="parent number x_loc y_loc z_loc">
@@ -96,16 +96,16 @@
     </link>
   </xacro:macro>
-<!--
+  <!--
     Stack macro - all the components relative transforms are made with respect
     to the parent link (usually base_link). They could be made relative to each
     other, but there is no necessary reason to do so.
   -->
- <xacro:macro name="stack_standard" params="parent">
-    <stack_bottom_pole parent="${parent}" number="0" x_loc= "0.1" y_loc= "0.115" z_loc="0.121"/>
-    <stack_bottom_pole parent="${parent}" number="1" x_loc= "-0.1" y_loc= "0.115" z_loc="0.121"/>
-    <stack_bottom_pole parent="${parent}" number="2" x_loc="0.1" y_loc= "-0.115" z_loc="0.121"/>
-    <stack_bottom_pole parent="${parent}" number="3" x_loc= "-0.1" y_loc="-0.115" z_loc="0.121"/>
-   <!-- bottom plate for Roch-->
-   <joint name="plate_bottom_joint" type="fixed">
+  <xacro:macro name="stack_standard" params="parent">
+    <xacro:stack_bottom_pole parent="${parent}" number="0" x_loc= "0.1" y_loc= "0.115" z_loc="0.121"/>
+    <xacro:stack_bottom_pole parent="${parent}" number="1" x_loc= "-0.1" y_loc= "0.115" z_loc="0.121"/>
+    <xacro:stack_bottom_pole parent="${parent}" number="2" x_loc="0.1" y_loc= "-0.115" z_loc="0.121"/>
+    <xacro:stack_bottom_pole parent="${parent}" number="3" x_loc= "-0.1" y_loc="-0.115" z_loc="0.121"/>
+    <!-- bottom plate for Roch-->
+    <joint name="plate_bottom_joint" type="fixed">
       <origin xyz="0 0.0 0.23" rpy="0 0 0"/>
       <parent link="base_link"/>
@@ -118,5 +118,5 @@
           <mesh filename="package://roch_description/meshes/stacks/plate_bottom.dae"/>
         </geometry>
-	<xacro:insert_block name="roch_dark_white"/>
+	      <xacro:insert_block name="roch_dark_white"/>
       </visual>
       <collision>
@@ -134,10 +134,10 @@
       </inertial>
     </link>
-    <stack_middle_pole parent="${parent}" number="0" x_loc= "0.1" y_loc= "0.115" z_loc="0.346"/>
-    <stack_middle_pole parent="${parent}" number="1" x_loc= "-0.1" y_loc= "0.115" z_loc="0.346"/>
-    <stack_middle_pole parent="${parent}" number="2" x_loc="0.1" y_loc= "-0.115" z_loc="0.346"/>
-    <stack_middle_pole parent="${parent}" number="3" x_loc= "-0.1" y_loc="-0.115" z_loc="0.346"/>
-   <!-- middle plate for Roch-->
-   <joint name="plate_middle_joint" type="fixed">
+    <xacro:stack_middle_pole parent="${parent}" number="0" x_loc= "0.1" y_loc= "0.115" z_loc="0.346"/>
+    <xacro:stack_middle_pole parent="${parent}" number="1" x_loc= "-0.1" y_loc= "0.115" z_loc="0.346"/>
+    <xacro:stack_middle_pole parent="${parent}" number="2" x_loc="0.1" y_loc= "-0.115" z_loc="0.346"/>
+    <xacro:stack_middle_pole parent="${parent}" number="3" x_loc= "-0.1" y_loc="-0.115" z_loc="0.346"/>
+    <!-- middle plate for Roch-->
+    <joint name="plate_middle_joint" type="fixed">
       <origin xyz="0 0.0 0.46" rpy="0 0 0"/>
       <parent link="base_link"/>
@@ -150,5 +150,5 @@
           <mesh filename="package://roch_description/meshes/stacks/plate_middle.dae"/>
         </geometry>
-	<xacro:insert_block name="roch_black"/>
+	      <xacro:insert_block name="roch_black"/>
       </visual>
       <collision>
@@ -166,9 +166,9 @@
       </inertial>
     </link>
-    <stack_top_pole parent="${parent}" number="0" x_loc="-0.16" y_loc= "0.0" z_loc="0.576"/>
-    <stack_top_pole parent="${parent}" number="1" x_loc="-0.13" y_loc= "0.06" z_loc="0.576"/>
-    <stack_top_pole parent="${parent}" number="2" x_loc="-0.13" y_loc= "-0.06" z_loc="0.576"/>
-<!-- sensor plate for Roch-->
-   <joint name="plate_sensor_joint" type="fixed">
+    <xacro:stack_top_pole parent="${parent}" number="0" x_loc="-0.16" y_loc= "0.0" z_loc="0.576"/>
+    <xacro:stack_top_pole parent="${parent}" number="1" x_loc="-0.13" y_loc= "0.06" z_loc="0.576"/>
+    <xacro:stack_top_pole parent="${parent}" number="2" x_loc="-0.13" y_loc= "-0.06" z_loc="0.576"/>
+    <!-- sensor plate for Roch-->
+    <joint name="plate_sensor_joint" type="fixed">
       <origin xyz="-0.14 0.0 0.691" rpy="0 0 0"/>
       <parent link="base_link"/>
@@ -181,10 +181,10 @@
           <mesh filename="package://roch_description/meshes/stacks/plate_sensor.dae"/>
         </geometry>
-	<xacro:insert_block name="roch_white"/>
+	      <xacro:insert_block name="roch_white"/>
       </visual>
       <collision>
         <origin xyz="-0.145 0.0 0.616" rpy="0 0 0"/>
         <geometry>
-           <box size="0.07 0.14 0.005"/>
+          <box size="0.07 0.14 0.005"/>
         </geometry>
       </collision>
